File: template/Full125Template/fx-Full125B.kicad_pcb (KiCad board)
At the start: 2 copper layers, 58 x 111.3 mm, 18 parts, among them J101 Conn_01x08_Pin, J102 Input, J103 Output, J104 Power

Commit message: Update Full 125B template
Parts:
- added TP101: TestPoint_Flag, TestPoint:TestPoint_Keystone_5000-5004_Miniature, F.Cu at (82.8, 50.8)
- added TP102: TestPoint_Flag, TestPoint:TestPoint_Keystone_5000-5004_Miniature, F.Cu at (119.5, 71.6)
- added TP103: TestPoint_Flag, TestPoint:TestPoint_Keystone_5000-5004_Miniature, F.Cu at (100.8, 71.6)
- added TP104: TestPoint_Flag, TestPoint:TestPoint_Keystone_5000-5004_Miniature, F.Cu at (137.2, 50.8)
- added TP105: TestPoint_Flag, TestPoint:TestPoint_Keystone_5000-5004_Miniature, F.Cu at (93.5, 132.2)
- added TP106: TestPoint_Flag, TestPoint:TestPoint_Keystone_5000-5004_Miniature, F.Cu at (126.5, 132.3)
- moved N101 84.0 mm to (137.6, 136.5), turned to 90 degrees
- moved D103 27.5 mm to (110.0, 125.6), turned to 180 degrees
- moved D104 24.3 mm to (110.0, 122.7), turned to 180 degrees
- moved D102 22.7 mm to (111.2, 127.9), turned to 180 degrees
- moved R105 19.2 mm to (120.0, 125.7), turned to 0 degrees
- moved R106 16.6 mm to (120.0, 124.2), turned to 0 degrees
- moved R104 14.7 mm to (120.0, 127.2), turned to 0 degrees
- moved J101 1.21 mm to (100.9, 132.3)
Connections:
- J101 pad 1: SENSE -> unconnected-(J101-Pin_1-Pad1)
- J101 pad 8: +9VA -> unconnected-(J101-Pin_8-Pad8)
Routing:
- net SW: track 35.8 -> 1.50 mm
- net +9VA: track 172.5 -> 145.6 mm
- net JACK_IN: track 114.2 -> 131.6 mm
- net +9V: track 12.9 -> 29.0 mm, vias 0 -> 1
- net EFFECT_OUT: track 0.00 -> 14.4 mm
- net EFFECT_IN: track 0.00 -> 14.1 mm
- net /Board Basic Setup/INT_PWR_LED: track 1.58 -> 8.86 mm
- net /Board Basic Setup/INT_SWITCH_LED: track 1.64 -> 8.14 mm
- net /Board Basic Setup/EXT_SWITCH_LED: track 3.62 -> 8.22 mm
- net GND: vias 33 -> 24
Other:
- board size 58 x 111.3 mm -> 58 x 100 mm
- board text added: "EIN"
- board text added: "FOOTSWITCH and LED Center on daughterboard -45mm ø 12.3mm"
- board text added: "Header Pin Centers for Footswitch Daughterboard"
- board text added: "LED Center (Above Footswitch) -27.4mm ø 5.2mm or 3.2mm"
- board text added: "LED Center (high, on PCB) -38mm ø 5.2mm or 3.2mm"
- board text added: "Pots/Switch center, go crazy with more than 6 holes"
- board text removed: "+9V"
- board text removed: "FOOTSWITCH CENTER -45mm ø 12.3mm"
- board text removed: "LED CENTER (high) -38mm ø 5.2mm or 3.2mm"
- board text removed: "LED CENTER (low) -45mm ø 5.2mm or 3.2mm"
- board text removed: "LFO"
- board text removed: "PIN"
