File: template/Full125Template/fx-Full125B.kicad_pcb (KiCad board)
At the start: 2 copper layers, 58 x 111.3 mm, 18 parts, among them J101 Conn_01x08_Pin, J102 Input, J103 Output, J104 Power

Commit message: Update Full-board 125B template.
Parts:
- added TP101: TestPoint_Flag, TestPoint:TestPoint_Keystone_5000-5004_Miniature, F.Cu at (86.6, 71.6)
- added TP102: TestPoint_Flag, TestPoint:TestPoint_Keystone_5000-5004_Miniature, F.Cu at (119.5, 71.6)
- added TP103: TestPoint_Flag, TestPoint:TestPoint_Keystone_5000-5004_Miniature, F.Cu at (100.8, 71.6)
- added TP104: TestPoint_Flag, TestPoint:TestPoint_Keystone_5000-5004_Miniature, F.Cu at (133.3, 71.5)
- added TP105: TestPoint_Flag, TestPoint:TestPoint_Keystone_5000-5004_Miniature, F.Cu at (93.5, 132.2)
- added TP106: TestPoint_Flag, TestPoint:TestPoint_Keystone_5000-5004_Miniature, F.Cu at (126.5, 132.3)
- J102, J103: footprint Effects_Footprints:Neutrik_NMJ6HCD2 -> Connector_Audio:Jack_6.35mm_Neutrik_NMJ6HCD2_Horizontal
- moved N101 84.0 mm to (137.6, 136.5), turned to 90 degrees
- moved D103 27.5 mm to (110.0, 125.6), turned to 180 degrees
- moved D104 24.3 mm to (110.0, 122.7), turned to 180 degrees
- moved D102 22.7 mm to (111.2, 127.9), turned to 180 degrees
- moved R105 19.2 mm to (120.0, 125.7), turned to 0 degrees
- moved R106 16.6 mm to (120.0, 124.2), turned to 0 degrees
- moved R104 14.7 mm to (120.0, 127.2), turned to 0 degrees
- moved C103 1.40 mm to (113.9, 72.5)
- moved C101 1.35 mm to (106.2, 72.5)
- moved J101 1.21 mm to (100.9, 132.3)
- moved J102 0.70 mm to (86.8, 61.5)
- moved J103 0.61 mm to (117.0, 61.4)
- moved J104 0.40 mm to (110.2, 53.5)
Connections:
- J101 pad 1: SENSE -> unconnected-(J101-Pin_1-Pad1)
- J101 pad 8: +9VA -> unconnected-(J101-Pin_8-Pad8)
Routing:
- net SW: track 35.8 -> 13.3 mm
- net +9VA: track 172.5 -> 152.7 mm
- net EFFECT_OUT: track 0.00 -> 14.4 mm
- net EFFECT_IN: track 0.00 -> 14.1 mm
- net JACK_IN: track 114.2 -> 121.6 mm
- net /Board Basic Setup/INT_PWR_LED: track 1.58 -> 8.86 mm
- net JACK_OUT: track 136.4 -> 129.3 mm
- net /Board Basic Setup/INT_SWITCH_LED: track 1.64 -> 8.14 mm
- net /Board Basic Setup/EXT_SWITCH_LED: track 3.62 -> 8.22 mm
- net +9V: track 12.9 -> 14.3 mm
- net GND: vias 33 -> 28
Other:
- board size 58 x 111.3 mm -> 58 x 100 mm
- board text added: "EIN"
- board text added: "FOOTSWITCH and LED Center on daughterboard -45mm ø 12.3mm"
- board text added: "Header Pin Centers for Footswitch Daughterboard"
- board text added: "LED Center (Above Footswitch) -27.4mm ø 5.2mm or 3.2mm"
- board text added: "LED Center (high, on PCB) -38mm ø 5.2mm or 3.2mm"
- board text added: "Pots/Switch center, go crazy with more than 6 holes"
- board text removed: "+9V"
- board text removed: "FOOTSWITCH CENTER -45mm ø 12.3mm"
- board text removed: "LED CENTER (high) -38mm ø 5.2mm or 3.2mm"
- board text removed: "LED CENTER (low) -45mm ø 5.2mm or 3.2mm"
- board text removed: "LFO"
- board text removed: "PIN"
