File: template/Full125Template/fx-Full125B.kicad_pcb (KiCad board)
At the start: 2 copper layers, 58 x 100 mm, 24 parts, among them J101 Conn_01x08_Pin, J102 Input, J103 Output, J104 Power

Commit message: Rework full template, add cap mult version
Parts:
- added D105: SMF24A, Diode_SMD:D_SMF, F.Cu at (107.3, 58.9)
- added D106: H5VU10BB, Diode_SMD:D_SOD-882, F.Cu at (83.0, 61.7)
- added D107: H15VL10B, Diode_SMD:D_SOD-882, F.Cu at (137.2, 61.5)
- added L101: GZ2012D601TF, Inductor_SMD:L_0805_2012Metric, F.Cu at (114.1, 64.6)
- J102, J103: footprint Connector_Audio:Jack_6.35mm_Neutrik_NMJ6HCD2_Horizontal -> Effects_Footprints:Neutrik_NMJ6HCD2
- R102, R103, R104, R105, R106: value 10k -> 10K
- moved R106 57.1 mm to (119.8, 67.1), turned to 90 degrees
- moved D104 55.9 mm to (118.2, 67.3), turned to -90 degrees
- moved TP101 20.4 mm to (83.1, 51.5), turned to 90 degrees
- moved TP104 20.3 mm to (136.8, 51.5)
- moved TP103 19.3 mm to (120.0, 73.1)
- moved TP102 19.2 mm to (100.4, 73.0)
- moved R103 9.26 mm to (105.6, 64.6)
- moved D101 8.98 mm to (113.0, 58.8), turned to 180 degrees
- moved R101 7.85 mm to (114.0, 61.3)
- moved C101 7.56 mm to (113.7, 71.2)
- moved C103 7.54 mm to (106.5, 71.2)
- moved R102 4.24 mm to (110.0, 66.2), turned to -90 degrees
- moved C102 1.65 mm to (110.0, 63.1)
Connections:
- D101 pad 1: +9VA -> Net-(D101-K)
- D101 pad 2: Net-(D101-A) -> +9V
- R101 pad 1: Net-(D101-A) -> Net-(FB101-Pad1)
- R101 pad 2: +9V -> Net-(D101-K)
Routing:
- net +9VA: track 152.7 -> 117.7 mm
- net JACK_IN: track 121.6 -> 90.7 mm
- net VREF: track 8.12 -> 0.00 mm
- net /Board Basic Setup/INT_PWR_LED: track 8.86 -> 2.33 mm
- net JACK_OUT: track 129.3 -> 123.9 mm, vias 0 -> 1
- net GND: track 0.00 -> 4.80 mm, vias 28 -> 56
- net +9V: track 14.3 -> 17.7 mm
- net Net-(D101-A): track 1.92 -> 0.00 mm
- net Net-(D101-K): track 0.00 -> 1.68 mm
- net Net-(FB101-Pad1): track 0.00 -> 1.47 mm
- net EFFECT_IN: track 14.1 -> 13.6 mm
- added copper zone on F.Cu, net JACK_IN
- added copper zone on F.Cu, net JACK_OUT
- added copper zone on F.Cu, net VREF
Other:
- board text added: "LED Center (high, on Daughterboard) -38mm ø 5.2mm or 3.2mm"
- board text added: "PedalName v0.1"
- board text added: "Y Centerline (0, 0 Tayda coords)"
- board text removed: "LED Center (high, on PCB) -38mm ø 5.2mm or 3.2mm"
- board text removed: "Y Centerline"
