File: template/Normal125B/Normal125B.kicad_pcb (KiCad board)
At the start: 2 copper layers, 50 x 50 mm, 13 parts, among them J101 Conn_01x03_Socket, J102 Conn_01x03_Socket

Commit message: Update: Some tweaks to the normal 125B template.
Other:
- board text added: "Max board Y dimension (footswitch clearance)"
- board text added: "NOTE: You can run 3-wide controls on a 50mm board if you castellate the pads, aligning them exactly half off the edge.cut! (Example alignment)"
