File: template/Normal125B/Normal125B.kicad_pcb (KiCad board)
At the start: 2 copper layers, 50 x 50 mm, 13 parts, among them J101 Conn_01x03_Socket, J102 Conn_01x03_Socket

Commit message: templates: consolidate all eight KiCad 10 templates in git, apply fleet kit v1
Canonical copies taken from ~/Documents/KiCad/10.0/template (what New Project has been instantiating).
Adds 1950XXFacePlate, BigFootTemplate, FullBoardChargePumpCapMult, PedalTemplate; drops backups, caches,
gerbers, lock files and the baked-in J102/J104 courtyard exclusions (now covered by the fleet jack rule).
Each template gains <name>.kicad_dru (fleet block), .gitignore, text defaults and component classes.
Normal125B board: 1049 insertions, 1105 deletions vs the stale repo copy (KiCad-folder version kept).

Co-Authored-By: Claude Fable 5.1 <noreply@anthropic.com>
Other:
- board text removed: "Max board Y dimension (footswitch clearance)"
- board text removed: "NOTE: You can run 3-wide controls on a 50mm board if you castellate the pads, aligning them exactly half off the edge.cut! (Example alignment)"
