File: template/Full125TemplateCapMult/board_setup.kicad_sch (KiCad schematic)
At the start: 28 parts, among them J101 Conn_01x08_Pin, J102 Input, J103 Output, J104 Power

Commit message: Rework full template, add cap mult version
Parts:
- removed C101: 100uF, Capacitor_SMD:CP_Elec_6.3x5.9, symbol Device:C_Polarized_Small_US
- removed C103: 100uF, Capacitor_SMD:CP_Elec_6.3x9.9, symbol Device:C_Polarized_Small_US
- removed D101: 1N5819, Diode_SMD:D_SOD-323, symbol Device:D_Small
- added C101, C106: 100n, Capacitor_SMD:C_0603_1608Metric, symbol Device:C_Small
- added C103, C107: 10u, Capacitor_SMD:C_1206_3216Metric, symbol Device:C_Small
- added C104: 100u, Capacitor_THT:CP_Radial_D6.3mm_P2.50mm, symbol Device:C_Polarized_Small_US
- added D101: 10V, Diode_SMD:D_SOD-123F, symbol Device:D_Zener_Small
- added Q101: AO3401A, Package_TO_SOT_SMD:SOT-23, symbol Transistor_FET:AO3401A
- added Q102: 2SC4212, Package_TO_SOT_SMD:SOT-23, symbol Transistor_BJT:2SC4213
- added R107: 100K, Resistor_SMD:R_0603_1608Metric, symbol Device:R_Small_US
- added U101: TL072, Package_SO:SOIC-8_3.9x4.9mm_P1.27mm, symbol Amplifier_Operational:TL072
- C102: value 100nF -> 10u; footprint Capacitor_SMD:C_0603_1608Metric -> Capacitor_SMD:C_1206_3216Metric
- R101: value 10R -> 10K; LCSC C22859 -> C25804
- R102: value 10K -> 1.2K
Connections:
- net +9V: now also L101.1
- net +9VA: now also R101.1, C106.1, Q102.2 (E), U101.8 (V+); no longer L101.2, R102.1
- net GND: now also C101.2, C103.2, C104.2, C106.2, C107.2, R107.2, U101.4 (V-)
- net VREF: now also U101.3 (+), U101.6 (-), U101.7; no longer R102.2, R103.1
- net at R101.2: now also R103.1, C107.1, U101.5 (+)
- new net: U101.1, U101.2 (-)
- new net: C103.1, C104.1, Q102.1 (B), R102.2
- new net: D101.2 (A), Q101.1 (G), R107.1
- new net: D101.1 (K), Q101.2 (S), Q102.3 (C), R102.1
- new net: C101.1, L101.2, Q101.3 (D)
Other:
- note added: "Cap multiplier (Q102): +9VA = Vrail − Vbe − (Iload/hFE)·R102 ← R102 sees only Iload/hFE Ripple rejection ≈ 1 / (2π·f·R102·Cbase) Cbase = C103 (+C104) → raise R102 and/or Cbase for more filtering; lower R102 only if (Iload/hFE)·R102 eats headroom (>~50 mA loads)"
- moved on the sheet: D105, J104, L101
