File: mn3102-dropin/clock_3102_cd4047.kicad_sch (KiCad schematic)
At the start: 5 parts, among them U1 CD4047B

Commit message: mn3102-dropin: SOIC-14 pads short the DIP-8 pins; switch adapter to TSSOP-14
SOIC-14 pad field reaches 3.45mm from centerline vs the DIP-8 pad ring
inner edge at 3.01mm (0.44mm overlap). TSSOP-14 rotated 90deg fits with
>=0.5mm clearance (2.15mm across). U1 footprint/LCSC now TSSOP-14
CD4047BPWR C2652491 (OOS at JLC/LCSC as of 2026-08-08: home-stencil from
Mouser/DigiKey, or overhang a SOIC on a stretched board); in-design use
keeps SOIC-14 C46538. ERC and golden netlist re-verified.

Co-Authored-By: Claude Fable 5 <noreply@anthropic.com>
Parts:
- U1: footprint Package_SO:SOIC-14_3.9x8.7mm_P1.27mm -> Package_SO:TSSOP-14_4.4x5mm_P0.65mm; LCSC C46538 -> C2652491
Changed lines of the file:
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@@
 			)
 		)
-		(property "Footprint" "Package_SO:SOIC-14_3.9x8.7mm_P1.27mm"
+		(property "Footprint" "Package_SO:TSSOP-14_4.4x5mm_P0.65mm"
 			(at 149.86 100.33 0)
 			(effects
@@
 			)
 		)
-		(property "Description" "CMOS monostable/astable multivibrator, wired astable as MN3102 replacement"
+		(property "Description" "TSSOP-14 rotated 90deg fits inside DIP-8 pin rows (adapter). For in-design JLC assembly use SOIC-14 CD4047BM96 LCSC C46538 instead."
 			(at 149.86 100.33 0)
 			(effects
@@
 			)
 		)
-		(property "LCSC" "C46538"
+		(property "LCSC" "C2652491"
 			(at 149.86 100.33 0)
 			(effects
@@
 		(instances
 			(project "fx-MN3102DropIn"
-				(path "/c7179315-4b50-4301-9663-fd6aac9515bd/eef4dae1-c24c-4d5f-937b-6697f15b36a4"
+				(path "/c556e1b7-f93a-4fb0-8141-9df2cef774de/95f8ed5c-c31d-4750-9045-e676dac2db76"
 					(reference "U1")
 					(unit 1)
@@
 		(instances
 			(project "fx-MN3102DropIn"
-				(path "/c7179315-4b50-4301-9663-fd6aac9515bd/eef4dae1-c24c-4d5f-937b-6697f15b36a4"
+				(path "/c556e1b7-f93a-4fb0-8141-9df2cef774de/95f8ed5c-c31d-4750-9045-e676dac2db76"
 					(reference "R1")
 					(unit 1)
@@
 		(instances
 			(project "fx-MN3102DropIn"
-				(path "/c7179315-4b50-4301-9663-fd6aac9515bd/eef4dae1-c24c-4d5f-937b-6697f15b36a4"
+				(path "/c556e1b7-f93a-4fb0-8141-9df2cef774de/95f8ed5c-c31d-4750-9045-e676dac2db76"
 					(reference "R2")
 					(unit 1)
@@
 		(instances
 			(project "fx-MN3102DropIn"
-				(path "/c7179315-4b50-4301-9663-fd6aac9515bd/eef4dae1-c24c-4d5f-937b-6697f15b36a4"
+				(path "/c556e1b7-f93a-4fb0-8141-9df2cef774de/95f8ed5c-c31d-4750-9045-e676dac2db76"
 					(reference "C1")
 					(unit 1)
@@
 		(instances
 			(project "fx-MN3102DropIn"
-				(path "/c7179315-4b50-4301-9663-fd6aac9515bd/eef4dae1-c24c-4d5f-937b-6697f15b36a4"
+				(path "/c556e1b7-f93a-4fb0-8141-9df2cef774de/95f8ed5c-c31d-4750-9045-e676dac2db76"
 					(reference "C2")
 					(unit 1)

Commit message: mn3102-dropin: shrink C2 to optional 100n 0603; all-top layout guidance
VGG draws no DC current, so C2 is filtering insurance only (100nF corner
~1.7kHz vs 50-200kHz clock); many hosts already cap the VGG net
(PizzaPizza C21 22uF). Was 1u 0805 (up to 1.25mm tall) - now 100n 0603
C14663, same part as C1, and DNP-able.

README: recommend all-top construction (~12.7mm board, TSSOP center,
0603s on end tongues, bare bottom, ~2.5mm overhang) - overhang verified
clear against fx-PizzaPizza placement (nearest on-axis parts are 0.8mm
0603s flying ~3.5mm below); bottom-side alternate needs collared pins.
0402 Basic alternates listed.

Co-Authored-By: Claude Fable 5 <noreply@anthropic.com>
Parts:
- C2: value 1u -> 100n; footprint Capacitor_SMD:C_0805_2012Metric -> Capacitor_SMD:C_0603_1608Metric; LCSC C28323 -> C14663
Changed lines of the file:
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@@
 			)
 		)
-		(property "Value" "1u"
+		(property "Value" "100n"
 			(at 191.77 93.98 0)
 			(effects
@@
 			)
 		)
-		(property "Footprint" "Capacitor_SMD:C_0805_2012Metric"
+		(property "Footprint" "Capacitor_SMD:C_0603_1608Metric"
 			(at 196.85 95.25 0)
 			(effects
@@
 			)
 		)
-		(property "LCSC" "C28323"
+		(property "LCSC" "C14663"
 			(at 196.85 95.25 0)
 			(effects
